Commit message: Resolved bugs in packet callbacks and added controller

File: bravo/config/urdf/bravo7.urdf (robot description, URDF)
Before this commit: robot bravo_7_example, 12 links, 11 joints
Links:
- added link ft_sensor_link, mass 0.05; visual cylinder length=0.041275 radius=0.0402
Joints:
- added joint ft_sensor_joint: type fixed, parent bravo_1023_0_joint_link, child ft_sensor_link, origin xyz=0.0408 -1.326794896676365e-09 -0.115 rpy=3.14159 -0.0 0.6, axis  0.  0. -1., limit lower=0.0 upper=6.2 effort=500.0 velocity=3.0
- joint bravo_axis_b: origin xyz=0.0408 -1.326794896676365e-09 -0.09434999999999824 rpy=3.14159 -0.0 0.6 -> xyz=0 0 0.020 rpy=0 -0.0 0.0; parent bravo_1023_0_joint_link -> ft_sensor_link
